Commit message: added apriltag

File: install/rmitbot_description/share/rmitbot_description/urdf/rmitbot.urdf.xacro (robot description, xacro)
@@ -1,13 +1 @@
-<?xml version="1.0"?>
-<!-- This is the main urdf document, calling other xacro, including -->
-<!-- rmitbot_platform:  main platform -->
-<!-- rmitbot_gazebo:    gazebo simulation parameters for the main platform -->
-<robot name="rmitbot"
-    xmlns:xacro="http://ros.org/wiki/xacro">
-    <xacro:include filename="$(find rmitbot_description)/urdf/rmitbot_platform.xacro" />
-    <xacro:include filename="$(find rmitbot_description)/urdf/rmitbot_gazebo.xacro" />
-    <xacro:include filename="$(find rmitbot_description)/urdf/rmitbot_ros2_control.xacro" />
-    <xacro:include filename="$(find rmitbot_description)/urdf/rmitbot_imu.xacro" />
-    <xacro:include filename="$(find rmitbot_description)/urdf/rmitbot_laser.xacro" />
-    <xacro:include filename="$(find rmitbot_description)/urdf/rmitbot_camera.xacro" />
-</robot>
+/home/v120506/rmitbot_v3/lesson6_ws/src/rmitbot_description/urdf/rmitbot.urdf.xacro

File: install/rmitbot_description/share/rmitbot_description/urdf/rmitbot_camera.xacro (robot description, xacro)
@@ -1,47 +1 @@
-<?xml version="1.0"?>
-<robot xmlns:xacro="http://www.ros.org/wiki/xacro" >
-    <joint name="camera_joint" type="fixed">
-        <parent link="base_link"/>
-        <child link="camera_link"/>
-        <origin xyz="0.15 0 0.08" rpy="0 0 0"/>
-    </joint>
-    <link name="camera_link">
-        <visual>
-            <geometry>
-                <box size="0.010 0.03 0.03"/>
-            </geometry>
-            <!-- <material name="red"/> -->
-        </visual>
-    </link>
-    <joint name="camera_optical_joint" type="fixed">
-        <parent link="camera_link"/>
-        <child link="camera_link_optical"/>
-        <origin xyz="0 0 0" rpy="${-pi/2} 0 ${-pi/2}"/>
-    </joint>
-    <link name="camera_link_optical"></link>
-    <gazebo reference="camera_link">
-        <!-- <material>Gazebo/Red</material> -->
-        <sensor name="camera" type="camera">
-            <pose> 0 0 0 0 0 0 </pose>
-            <visualize>true</visualize>
-            <always_on>true</always_on>
-            <update_rate>10</update_rate>
-            <camera>
-                <horizontal_fov>1.089</horizontal_fov>
-                <image>
-                    <format>R8G8B8</format>
-                    <width>640</width>
-                    <height>480</height>
-                </image>
-                <clip>
-                    <near>0.05</near>
-                    <far>8.0</far>
-                </clip>
-            </camera>
-            <topic>/camera/image</topic>
-            <!-- <plugin name="camera_controller" filename="libgazebo_ros_camera.so">
-                <frame_name>camera_link_optical</frame_name>
-            </plugin> -->
-        </sensor>
-    </gazebo>
-</robot>
+/home/v120506/rmitbot_v3/lesson6_ws/src/rmitbot_description/urdf/rmitbot_camera.xacro

File: install/rmitbot_description/share/rmitbot_description/urdf/rmitbot_gazebo.xacro (robot description, xacro)
@@ -1,63 +1 @@
-<?xml version="1.0"?>
-<!-- Gazebo file contains information regarding the lnks's physics (e.g., friction, stiffness, damping) -->
-<robot name="rmitbot" xmlns:xacro="http://ros.org/wiki/xacro" xmlns:gz="http://gazebosim.org/schema">
-  <!-- Wheels -->
-     <!-- To emulate Mecanum wheels in Gazebo with spherical collisions it
-  requires a custom friction model so the vehicle can strafe left to right -->
-  <gazebo reference='front_left_wheel'>
-    <collision>
-      <surface>
-        <friction>
-          <ode>
-            <mu>1.0</mu>
-            <mu2>0.0</mu2>
-            <!-- <fdir1 gz:expressed_in="base_link">1 -1 0</fdir1> -->
-            <fdir1 gz:expressed_in="base_footprint">1 -1 0</fdir1>
-          </ode>
-        </friction>
-      </surface>
-    </collision>
-  </gazebo>
-  <gazebo reference='front_right_wheel'>
-    <collision>
-      <surface>
-        <friction>
-          <ode>
-            <mu>1.0</mu>
-            <mu2>0.0</mu2>
-            <!-- <fdir1 gz:expressed_in="base_link">1 1 0</fdir1> -->
-            <fdir1 gz:expressed_in="base_footprint">1 1 0</fdir1>
-          </ode>
-        </friction>
-      </surface>
-    </collision>
-  </gazebo>
-  <gazebo reference='rear_left_wheel'>
-    <collision>
-      <surface>
-        <friction>
-          <ode>
-            <mu>1.0</mu>
-            <mu2>0.0</mu2>
-            <!-- <fdir1 gz:expressed_in="base_link">1 1 0</fdir1> -->
-            <fdir1 gz:expressed_in="base_footprint">1 1 0</fdir1>
-          </ode>
-        </friction>
-      </surface>
-    </collision>
-  </gazebo>
-  <gazebo reference='rear_right_wheel'>
-    <collision>
-      <surface>
-        <friction>
-          <ode>
-            <mu>1.0</mu>
-            <mu2>0.0</mu2>
-            <!-- <fdir1 gz:expressed_in="base_link">1 -1 0</fdir1> -->
-            <fdir1 gz:expressed_in="base_footprint">1 -1 0</fdir1>
-          </ode>
-        </friction>
-      </surface>
-    </collision>
-  </gazebo>
-</robot>
+/home/v120506/rmitbot_v3/lesson6_ws/src/rmitbot_description/urdf/rmitbot_gazebo.xacro

File: install/rmitbot_description/share/rmitbot_description/urdf/rmitbot_imu.xacro (robot description, xacro)
@@ -1,88 +1 @@
-<?xml version="1.0"?>
-<robot xmlns:xacro="http://www.ros.org/wiki/xacro" name="rmitbot">
-    <link name="imu_link">
-        <inertial>
-            <origin xyz="-0.0055 0.00017 0.00051" rpy="0 0 0" />
-            <mass value="0.00053" />
-            <inertia  ixx="1.46E-08" ixy="1.40E-10" ixz="-1.99E-12"
-                      iyy="8.59E-09" iyz="7.52E-12" izz="2.30E-08" />
-        </inertial>
-        <visual>
-            <origin xyz="0 0 0" rpy="0 0 0" />
-            <geometry>
-                <mesh filename="package://rmitbot_description/meshes/imu_link.STL" />
-            </geometry>
-            <material name="">
-                <color rgba="0.8 0.8 0.94 1" />
-            </material>
-        </visual>
-        <collision>
-            <origin xyz="0 0 0" rpy="0 0 0" />
-            <geometry>
-                <mesh filename="package://rmitbot_description/meshes/imu_link.STL" />
-            </geometry>
-        </collision>
-    </link>
-    <joint name="imu_joint" type="fixed">
-        <origin xyz="0 0 0.1" rpy="0 0 0" />
-        <parent link="base_link" />
-        <child link="imu_link" />
-        <axis xyz="0 0 0" />
-    </joint>
-    <!-- Gazebo plugins for IMU-->
-    <gazebo>
-        <plugin filename="gz-sim-imu-system" name="gz::sim::systems::Imu">
-        </plugin>
-    </gazebo>
-    <!-- Gazebo parameters for IMU, with noise-->
-  <gazebo reference="imu_link">
-    <sensor name="imu" type="imu">
-      <always_on>true</always_on>
-      <update_rate>100</update_rate>
-      <gz_frame_id>imu_link</gz_frame_id>
-      <topic>imu</topic>
-      <imu>
-        <angular_velocity>
-          <x>
-            <noise type="gaussian">
-              <mean>0.0</mean>
-              <stddev>2e-4</stddev>
-            </noise>
-          </x>
-          <y>
-            <noise type="gaussian">
-              <mean>0.0</mean>
-              <stddev>2e-4</stddev>
-            </noise>
-          </y>
-          <z>
-            <noise type="gaussian">
-              <mean>0.0</mean>
-              <stddev>2e-4</stddev>
-            </noise>
-          </z>
-        </angular_velocity>
-        <linear_acceleration>
-          <x>
-            <noise type="gaussian">
-              <mean>0.0</mean>
-              <stddev>1.7e-2</stddev>
-            </noise>
-          </x>
-          <y>
-            <noise type="gaussian">
-              <mean>0.0</mean>
-              <stddev>1.7e-2</stddev>
-            </noise>
-          </y>
-          <z>
-            <noise type="gaussian">
-              <mean>0.0</mean>
-              <stddev>1.7e-2</stddev>
-            </noise>
-          </z>
-        </linear_acceleration>
-      </imu>
-    </sensor>
-  </gazebo>
-</robot>
+/home/v120506/rmitbot_v3/lesson6_ws/src/rmitbot_description/urdf/rmitbot_imu.xacro

File: install/rmitbot_description/share/rmitbot_description/urdf/rmitbot_laser.xacro (robot description, xacro)
@@ -1,70 +1 @@
-<?xml version="1.0"?>
-<robot xmlns:xacro="http://www.ros.org/wiki/xacro" name="rmitbot">
-    <link name="laser_link">
-        <inertial>
-            <origin xyz="-0.012 -0.00038 -0.017" rpy="0 0 0" />
-            <mass value="0.073" />
-            <inertia    ixx="1.96E-05" ixy="-3.62E-07" ixz="4.28E-07"
-                        iyy="2.41E-05" iyz="1.50E-08" izz="4.14E-05" />
-        </inertial>
-        <visual>
-            <origin xyz="0 0 0" rpy="0 0 0" />
-            <geometry>
-                <mesh filename="package://rmitbot_description/meshes/laser_link.STL" />
-            </geometry>
-        </visual>
-        <collision>
-            <origin xyz="0 0 0" rpy="0 0 0" />
-            <geometry>
-                <mesh filename="package://rmitbot_description/meshes/laser_link.STL" />
-            </geometry>
-        </collision>
-    </link>
-    <joint name="laser_joint" type="fixed">
-        <origin xyz="0. 0. 0.14" rpy="0 0 3.14" />
-        <parent link="base_link" />
-        <child link="laser_link" />
-        <axis xyz="0 0 0" />
-    </joint>
-    <gazebo reference="laser_link">
-        <sensor name="lidar" type="gpu_lidar">
-            <!-- <sensor name="lidar" type="ray"> -->
-            <plugin filename="gz-sim-sensors-system" name="gz::sim::systems::Sensors">
-                <render_engine>ogre</render_engine>
-            </plugin>
-            <always_on>true</always_on>
-            <visualize>true</visualize>
-            <topic>scan</topic>
-            <update_rate>5</update_rate>
-            <gz_frame_id>laser_link</gz_frame_id>
-            <lidar>
-                <!-- <ray> -->
-                <scan>
-                    <horizontal>
-                        <samples>360</samples>
-                        <resolution>1.00000</resolution>
-                        <min_angle>0.000000</min_angle>
-                        <max_angle>6.280000</max_angle>
-                    </horizontal>
-                    <!-- Dirty hack for fake lidar detections with ogre 1 rendering in VM -->
-                    <vertical>
-                        <samples>3</samples>
-                        <min_angle>-0.001</min_angle>
-                        <max_angle>0.001</max_angle>
-                    </vertical>
-                </scan>
-                <range>
-                    <min>0.120000</min>
-                    <max>12.0</max>
-                    <resolution>0.02</resolution>
-                </range>
-                <noise>
-                    <type>gaussian</type>
-                    <mean>0.0</mean>
-                    <stddev>0.01</stddev>
-                </noise>
-            </lidar>
-            <!-- </ray> -->
-        </sensor>
-    </gazebo>
-</robot>
+/home/v120506/rmitbot_v3/lesson6_ws/src/rmitbot_description/urdf/rmitbot_laser.xacro

File: install/rmitbot_description/share/rmitbot_description/urdf/rmitbot_platform.xacro (robot description, xacro)
@@ -1,189 +1 @@
-<?xml version="1.0"?>
-<robot name="rmitbot" xmlns:xacro="http://www.ros.org/wiki/xacro" xmlns:gz="http://gazebosim.org/schema">
-  <material name="orange">
-    <color rgba="0.8 0.4 0.0 1.0" />
-  </material>
-  <material name="black">
-    <color rgba="0.5 0.5 0.5 1.0" />
-  </material>
-  <material name="white">
-    <color rgba="1 1 1 1.0" />
-  </material>
-  <link name="base_footprint" />
-  <joint name="base_joint" type="fixed">
-    <parent link="base_footprint" />
-    <child link="base_link" />
-    <origin xyz="0 0 0.05" rpy="0 0 0" />
-  </joint>
-  <!-- Base Link -->
-  <link name="base_link">
-    <collision>
-      <origin xyz="0 0 0.05" rpy="0 0 0" />
-      <geometry>
-         <box size=".28 .3 0.1" />
-      </geometry>
-    </collision>
-    <visual>
-      <origin xyz="0 0 0.05" rpy="0 0 0" />
-      <geometry>
-         <box size=".28 .3 0.1" />
-      </geometry>
-      <material name="orange" />
-    </visual>
-    <inertial>
-      <origin xyz="0 0 0.5" rpy="0 0 0" />
-      <mass value="1.5" />
-      <inertia
-        ixx="0.13"
-        ixy="0.0"
-        ixz="0.0"
-        iyy="0.42"
-        iyz="0.0"
-        izz="0.48" />
-    </inertial>
-  </link>
-  <!-- front left wheel -->
-  <joint name="front_left_wheel_joint" type="continuous">
-    <origin xyz="0.14 0.15 0" rpy="-${pi/2} 0 0" />
-    <parent link="base_link" />
-    <child link="front_left_wheel" />
-    <axis xyz="0 0 1" />
-    <dynamics damping="0.2" />
-  </joint>
-  <link name="front_left_wheel">
-    <collision>
-      <!-- <origin xyz="0 0 .06" rpy="0 0 0" /> -->
-      <origin xyz="0 0 .025" rpy="0 0 0" />
-      <geometry>
-        <sphere radius="0.05" />
-      </geometry>
-    </collision>
-    <visual>
-      <!-- <origin xyz="0 0 .06" rpy="0 0 0" /> -->
-      <origin xyz="0 0 .025" rpy="0 0 0" />
-      <geometry>
-        <!-- <sphere radius="0.3" /> -->
-        <cylinder radius="0.05" length="0.05" />
-      </geometry>
-      <material name="black" />
-    </visual>
-    <inertial>
-      <!-- <origin xyz="0 0 .06" rpy="0 0 0" /> -->
-       <origin xyz="0 0 .025" rpy="0 0 0" />
-      <mass value="0.5" />
-      <inertia ixx="0.0025"
-        ixy="0.0"
-        ixz="0.0"
-        iyy="0.0025"
-        iyz="0.0"
-        izz="0.0020" />
-    </inertial>
-  </link>
-  <!-- front right wheel -->
-  <joint name="front_right_wheel_joint" type="continuous">
-    <origin xyz="0.14 -0.15 0." rpy="-${pi/2} 0 0" />
-    <parent link="base_link" />
-    <child link="front_right_wheel" />
-    <axis xyz="0 0 1" />
-    <dynamics damping="0.2" />
-  </joint>
-  <link name="front_right_wheel">
-    <collision>
-      <!-- <origin xyz="0 0 -.06" rpy="0 0 0" /> -->
-      <origin xyz="0 0 -.025" rpy="0 0 0" />
-      <geometry>
-        <sphere radius="0.05" />
-      </geometry>
-    </collision>
-    <visual>
-      <origin xyz="0 0 -.025" rpy="0 0 0" />
-      <geometry>
-        <cylinder radius="0.05" length="0.05" />
-      </geometry>
-      <material name="black" />
-    </visual>
-    <inertial>
-      <!-- <origin xyz="0 0 -.06" rpy="0 0 0" /> -->
-      <origin xyz="0 0 -.025" rpy="0 0 0" />
-      <mass value=".5" />
-      <inertia ixx="0.0025"
-        ixy="0.0"
-        ixz="0.0"
-        iyy="0.0025"
-        iyz="0.0"
-        izz="0.0020" />
-    </inertial>
-  </link>
-  <!-- rear left wheel -->
-  <joint name="rear_left_wheel_joint" type="continuous">
-    <origin xyz="-0.14 0.15 0." rpy="-${pi/2} 0 0" />
-    <parent link="base_link" />
-    <child link="rear_left_wheel" />
-    <axis xyz="0 0 1" />
-    <dynamics damping="0.2" />
-  </joint>
-  <link name="rear_left_wheel">
-    <collision>
-      <!-- <origin xyz="0 0 .06" rpy="0 0 0" /> -->
-       <origin xyz="0 0 .025" rpy="0 0 0" />
-      <geometry>
-        <sphere radius="0.05" />
-      </geometry>
-    </collision>
-    <visual>
-      <!-- <origin xyz="0 0 .06" rpy="0 0 0" /> -->
-       <origin xyz="0 0 .025" rpy="0 0 0" />
-      <geometry>
-        <cylinder radius="0.05" length="0.05" />
-      </geometry>
-      <material name="black" />
-    </visual>
-    <inertial>
-      <!-- <origin xyz="0 0 .06" rpy="0 0 0" /> -->
-       <origin xyz="0 0 .025" rpy="0 0 0" />
-      <mass value="0.5" />
-      <inertia ixx="0.0025"
-        ixy="0.0"
-        ixz="0.0"
-        iyy="0.0025"
-        iyz="0.0"
-        izz="0.0020" />
-    </inertial>
-  </link>
-  <!-- rear right wheel -->
-  <joint name="rear_right_wheel_joint" type="continuous">
-    <origin xyz="-0.14 -0.15 0." rpy="-${pi/2} 0 0" />
-    <parent link="base_link" />
-    <child link="rear_right_wheel" />
-    <axis xyz="0 0 1" />
-    <dynamics damping="0.2" />
-  </joint>
-  <link name="rear_right_wheel">
-    <collision>
-      <!-- <origin xyz="0 0 -.06" rpy="0 0 0" /> -->
-       <origin xyz="0 0 -.025" rpy="0 0 0" />
-      <geometry>
-        <sphere radius="0.05" />
-      </geometry>
-    </collision>
-    <visual>
-      <!-- <origin xyz="0 0 -.06" rpy="0 0 0" /> -->
-       <origin xyz="0 0 -.025" rpy="0 0 0" />
-      <geometry>
-        <cylinder radius="0.05" length="0.05" />
-      </geometry>
-      <material name="black" />
-    </visual>
-    <inertial>
-      <!-- <origin xyz="0 0 -.06" rpy="0 0 0" /> -->
-       <origin xyz="0 0 -.025" rpy="0 0 0" />
-      <mass value="0.5" />
-      <inertia ixx="0.0025"
-        ixy="0.0"
-        ixz="0.0"
-        iyy="0.0025"
-        iyz="0.0"
-        izz="0.0020" />
-    </inertial>
-  </link>
-</robot>
+/home/v120506/rmitbot_v3/lesson6_ws/src/rmitbot_description/urdf/rmitbot_platform.xacro

File: install/rmitbot_description/share/rmitbot_description/urdf/rmitbot_ros2_control.xacro (robot description, xacro)
@@ -1,49 +1 @@
-<?xml version="1.0"?>
-<robot name="rmitbot" xmlns:xacro="http://www.ros.org/wiki/xacro"> Define the vehicles hardware,
-    command and state interfaces <ros2_control name="GazeboSimSystem" type="system">
-        <hardware>
-            <plugin>gz_ros2_control/GazeboSimSystem</plugin>
-        </hardware>
-        <joint name="front_left_wheel_joint">
-            <command_interface name="velocity">
-                <param name="min">-1</param>
-                <param name="max">1</param>
-            </command_interface>
-            <state_interface name="position" />
-            <state_interface name="velocity" />
-        </joint>
-        <joint name="front_right_wheel_joint">
-            <command_interface name="velocity">
-                <param name="min">-1</param>
-                <param name="max">1</param>
-            </command_interface>
-            <state_interface name="position" />
-            <state_interface name="velocity" />
-        </joint>
-        <joint name="rear_left_wheel_joint">
-            <command_interface name="velocity">
-                <param name="min">-1</param>
-                <param name="max">1</param>
-            </command_interface>
-            <state_interface name="position" />
-            <state_interface name="velocity" />
-        </joint>
-        <joint name="rear_right_wheel_joint">
-            <command_interface name="velocity">
-                <param name="min">-1</param>
-                <param name="max">1</param>
-            </command_interface>
-            <state_interface name="position" />
-            <state_interface name="velocity" />
-        </joint>
-    </ros2_control>
-    <!-- ROS2 Control plugin and topic re-mapping -->
-  <gazebo>
-        <plugin filename="gz_ros2_control-system" name="gz_ros2_control::GazeboSimROS2ControlPlugin">
-            <parameters>$(find rmitbot_controller)/config/rmitbot_controller.yaml</parameters>
-            <ros>
-                <remapping>/mecanum_drive_controller/odom:=/odom</remapping>
-            </ros>
-        </plugin>
-    </gazebo>
-</robot>
+/home/v120506/rmitbot_v3/lesson6_ws/src/rmitbot_description/urdf/rmitbot_ros2_control.xacro

File: src/rmitbot_description/urdf/rmitbot_camera.xacro (robot description, xacro)
@@ -1,13 +1,13 @@
 <?xml version="1.0"?>
-<robot xmlns:xacro="http://www.ros.org/wiki/xacro" >
+<robot xmlns:xacro="http://www.ros.org/wiki/xacro">
     <joint name="camera_joint" type="fixed">
-        <parent link="base_link"/>
-        <child link="camera_link"/>
-        <origin xyz="0.15 0 0.08" rpy="0 0 0"/>
+        <parent link="base_link" />
+        <child link="camera_link" />
+        <origin xyz="0.15 0 0.08" rpy="0 0 0" />
     </joint>
     <link name="camera_link">
         <visual>
             <geometry>
-                <box size="0.010 0.03 0.03"/>
+                <box size="0.010 0.03 0.03" />
             </geometry>
             <!-- <material name="red"/> -->
@@ -15,16 +15,17 @@
     </link>
     <joint name="camera_optical_joint" type="fixed">
-        <parent link="camera_link"/>
-        <child link="camera_link_optical"/>
-        <origin xyz="0 0 0" rpy="${-pi/2} 0 ${-pi/2}"/>
+        <parent link="camera_link" />
+        <child link="camera_link_optical" />
+        <origin xyz="0 0 0" rpy="${-pi/2} 0 ${-pi/2}" />
     </joint>
     <link name="camera_link_optical"></link>
     <gazebo reference="camera_link">
-        <!-- <material>Gazebo/Red</material> -->
         <sensor name="camera" type="camera">
-            <pose> 0 0 0 0 0 0 </pose>
             <visualize>true</visualize>
             <always_on>true</always_on>
-            <update_rate>10</update_rate>
+            <update_rate>20</update_rate>
+            <topic>/camera/image</topic>
+            <pose> 0 0 0 0 0 0 </pose>
+            <gz_frame_id>camera_link_optical</gz_frame_id>
             <camera>
                 <horizontal_fov>1.089</horizontal_fov>
@@ -38,9 +39,6 @@
                     <far>8.0</far>
                 </clip>
+                <camera_info_topic>camera/camera_info</camera_info_topic>
             </camera>
-            <topic>/camera/image</topic>
-            <!-- <plugin name="camera_controller" filename="libgazebo_ros_camera.so">
-                <frame_name>camera_link_optical</frame_name>
-            </plugin> -->
         </sensor>
     </gazebo>
